Commit message: modify ground truth plugin

File: scout_gazebo/urdf/base.xacro (robot description, xacro)
@@ -19,19 +19,4 @@
         <color rgba="0.0 0.0 0.0 1.0" />
     </material>
-    <!--插件-->
-    <!--xacro:include
-    filename ="$(find scout_gazebo)/urdf/plugin.xacro" -->
-    <gazebo>
-        <plugin name="ground_truth" filename="libgazebo_ros_p3d.so">
-            <alwaysOn>true</alwaysOn>
-            <updateRate>50.0</updateRate>
-            <bodyName>base_link</bodyName>
-            <topicName>base_pose_ground_truth</topicName>
-            <gaussianNoise>0.0</gaussianNoise>
-            <frameName>map</frameName>
-            <xyzOffsets>0 0 0</xyzOffsets>
-            <rpyOffsets>0 0 0</rpyOffsets>
-        </plugin>
-    </gazebo>
     <!-- 底盘的轮子 -->
     <xacro:include filename="$(find scout_gazebo)/urdf/scout_wheel_type1.xacro" />
@@ -45,18 +30,29 @@
         <origin rpy="0 0 0" xyz="0 0 0.3" />
     </xacro:realsense_d435> -->
+    <xacro:include filename="$(find scout_gazebo)/urdf/laser_support.xacro" />
     <!-- VLP16 激光雷达 -->
-    <xacro:include filename="$(find scout_gazebo)/urdf/laser_support.xacro" />
     <!-- <xacro:include filename="$(find velodyne_description)/urdf/VLP-16.urdf.xacro"/>
-    <xacro:VLP-16 parent="support" name="velodyne" topic="/scan" organize_cloud="${organize_cloud}"
+    <xacro:VLP-16 parent="support" name="lidar" topic="/scan" organize_cloud="${organize_cloud}"
     hz="10" samples="1800" max_range="150" gpu="${gpu}">
-          <origin xyz="0 0 ${support_length/2}" rpy="0 0 0" />
+          <origin xyz="0 0 0" rpy="0 0 0" />
     </xacro:VLP-16> -->
+    <!-- 车载120°激光雷达 -->
+    <!-- <xacro:include filename="$(find velodyne_description)/urdf/Lidar.urdf.xacro" />
+    <xacro:Lidar parent="support" name="lidar" topic="/scan" hz="10"
+        organize_cloud="${organize_cloud}" gpu="${gpu}"
+        samples="480" min_horizonal_angle="-${60.0*M_PI/180.0}" max_horizonal_angle="${60.0*M_PI/180.0}"
+        lasers="96" min_vertical_angle="-${12.5*M_PI/180.0}" max_vertical_angle="${12.5*M_PI/180.0}">
+        <origin xyz="0 0 0" rpy="0 0 0" />
+    </xacro:Lidar> -->
+    <!-- Livox Avia激光雷达 -->
     <xacro:include filename="$(find livox_laser_simulation)/urdf/livox_avia.xacro" />
-    <xacro:Livox_AVIA name="livox" parent="support" />
+    <xacro:Livox_Avia name="lidar" parent="support" />
     <!-- IMU 模块 -->
     <xacro:include filename="$(find scout_gazebo)/urdf/imu.xacro" />
-    <xacro:imu sensor_name="imu" parent_link="base_link">
+    <xacro:imu sensor_name="imu" parent_link="lidar">
         <origin rpy="0 0 0" xyz="0 0 0" />
     </xacro:imu>
+    <!--真值插件-->
+    <xacro:include filename ="$(find scout_gazebo)/urdf/ground_truth.xacro" />
     <!-- 机器人导航控制模块 -->
     <xacro:include filename="$(find scout_gazebo)/urdf/move.xacro" />

File: scout_gazebo/urdf/imu.xacro (robot description, xacro)
@@ -12,7 +12,7 @@
             <xacro:insert_block name="origin" />
             <parent link="${parent_link}"/>
-            <child link="imu_base"/>
+            <child link="imu"/>
         </joint>
-        <link name="imu_base">
+        <link name="imu">
             <visual>
                 <origin rpy="0 0 0" xyz="0 0 0" />
@@ -33,5 +33,5 @@
         </link>
         <!-- 被引用的link -->
-        <gazebo reference="imu_base">
+        <gazebo reference="imu">
             <material>Gazebo/Bule</material>
             <gravity>true</gravity>
@@ -43,10 +43,10 @@
             <plugin filename="libgazebo_ros_imu_sensor.so" name="imu_plugin">
                 <topicName>imu/data</topicName>
-                <bodyName>imu_base</bodyName>
+                <bodyName>imu</bodyName>
                 <updateRateHZ>200.0</updateRateHZ>
                 <gaussianNoise>0.01</gaussianNoise>
                 <xyzOffset>0 0 0</xyzOffset>
                 <rpyOffset>0 0 0</rpyOffset>
-                <frameName>imu_base</frameName>
+                <frameName>imu</frameName>
             </plugin>
             <pose>0 0 0 0 0 0</pose>

Commit message: add choice of lidar type in xacro

File: scout_gazebo/urdf/base.xacro (robot description, xacro)
@@ -3,5 +3,7 @@
     <xacro:arg name="robot_namespace" default="/" />
     <!-- 属性封装 -->
-    <xacro:property name="M_PI" value="3.14159" />
+    <!-- 0 for velodyne, 1 for livox, 2 for 120*25 solid lidar -->
+    <xacro:arg name="lidar_type" default="2" />
+    <xacro:property name="lidar_type" value="$(arg lidar_type)" />
     <xacro:property name="base_x_size" value="0.9250000" />
     <xacro:property name="base_y_size" value="0.380000" />
@@ -31,21 +33,28 @@
     </xacro:realsense_d435> -->
     <xacro:include filename="$(find scout_gazebo)/urdf/laser_support.xacro" />
-    <!-- VLP16 激光雷达 -->
-    <!-- <xacro:include filename="$(find velodyne_description)/urdf/VLP-16.urdf.xacro"/>
-    <xacro:VLP-16 parent="support" name="lidar" topic="/scan" organize_cloud="${organize_cloud}"
-    hz="10" samples="1800" max_range="150" gpu="${gpu}">
-          <origin xyz="0 0 0" rpy="0 0 0" />
-    </xacro:VLP-16> -->
-    <!-- 车载120°激光雷达 -->
-    <!-- <xacro:include filename="$(find velodyne_description)/urdf/Lidar.urdf.xacro" />
-    <xacro:Lidar parent="support" name="lidar" topic="/scan" hz="10"
-        organize_cloud="${organize_cloud}" gpu="${gpu}"
-        samples="480" min_horizonal_angle="-${60.0*M_PI/180.0}" max_horizonal_angle="${60.0*M_PI/180.0}"
-        lasers="96" min_vertical_angle="-${12.5*M_PI/180.0}" max_vertical_angle="${12.5*M_PI/180.0}">
-        <origin xyz="0 0 0" rpy="0 0 0" />
-    </xacro:Lidar> -->
-    <!-- Livox Avia激光雷达 -->
-    <xacro:include filename="$(find livox_laser_simulation)/urdf/livox_avia.xacro" />
-    <xacro:Livox_Avia name="lidar" parent="support" />
+    <!-- ${}里可以使用python语句 -->
+    <xacro:if value="${lidar_type==0}">
+        <!-- VLP16 激光雷达 -->
+        <xacro:include filename="$(find velodyne_description)/urdf/VLP-16.urdf.xacro"/>
+        <xacro:VLP-16 parent="support" name="lidar" topic="/scan" organize_cloud="${organize_cloud}"
+        hz="10" samples="1800" max_range="150" gpu="${gpu}">
+              <origin xyz="0 0 0" rpy="0 0 0" />
+        </xacro:VLP-16>
+    </xacro:if>
+    <xacro:if value="${lidar_type==1}">
+        <!-- Livox Avia激光雷达 -->
+        <xacro:include filename="$(find livox_laser_simulation)/urdf/livox_avia.xacro" />
+        <xacro:Livox_Avia name="lidar" parent="support" />
+    </xacro:if>
+    <xacro:if value="${lidar_type==2}">
+        <!-- 车载120°激光雷达 -->
+        <xacro:include filename="$(find velodyne_description)/urdf/Lidar.urdf.xacro" />
+        <xacro:Lidar parent="support" name="lidar" topic="/scan" hz="10"
+            organize_cloud="${organize_cloud}" gpu="${gpu}"
+            samples="480" min_horizonal_angle="${radians(-60.0)}" max_horizonal_angle="${radians(60.0)}"
+            lasers="96" min_vertical_angle="${radians(-12.5)}" max_vertical_angle="${radians(12.5)}">
+            <origin xyz="0 0 0" rpy="0 0 0" />
+        </xacro:Lidar>
+    </xacro:if>
     <!-- IMU 模块 -->
     <xacro:include filename="$(find scout_gazebo)/urdf/imu.xacro" />
@@ -96,5 +105,5 @@
     <!-- motor 1 and 2 (left side) are mechanically installed in a reversed direction -->
     <xacro:scout_wheel_type1 wheel_prefix="front_right">
-        <origin xyz="${wheelbase/2} ${-track/2} ${wheel_vertical_offset}" rpy="3.14 0 0" />
+        <origin xyz="${wheelbase/2} ${-track/2} ${wheel_vertical_offset}" rpy="${radians(180)} 0 0" />
     </xacro:scout_wheel_type1>
     <xacro:scout_wheel_type2 wheel_prefix="front_left">
@@ -105,5 +114,5 @@
     </xacro:scout_wheel_type1>
     <xacro:scout_wheel_type2 wheel_prefix="rear_right">
-        <origin xyz="${-wheelbase/2} ${-track/2} ${wheel_vertical_offset}" rpy="3.14 0 0" />
+        <origin xyz="${-wheelbase/2} ${-track/2} ${wheel_vertical_offset}" rpy="${radians(180)} 0 0" />
     </xacro:scout_wheel_type2>
 </robot>

File: scout_gazebo/urdf/scout_wheel_type1.xacro (robot description, xacro)
@@ -38,5 +38,5 @@
             </visual>
             <collision>
-                <origin xyz="0 0 0" rpy="${M_PI/2} 0 0" />
+                <origin xyz="0 0 0" rpy="${radians(90)} 0 0" />
                 <geometry>
                     <cylinder length="${wheel_length}" radius="${wheel_radius}" />

File: scout_gazebo/urdf/scout_wheel_type2.xacro (robot description, xacro)
@@ -38,5 +38,5 @@
             </visual>
             <collision>
-                <origin xyz="0 0 0" rpy="${M_PI/2} 0 0" />
+                <origin xyz="0 0 0" rpy="${radians(90)} 0 0" />
                 <geometry>
                     <cylinder length="${wheel_length}" radius="${wheel_radius}" />

Commit message: modify the sequence of elements in velodyne msg

File: scout_gazebo/urdf/base.xacro (robot description, xacro)
@@ -4,5 +4,5 @@
     <!-- 属性封装 -->
     <!-- 0 for velodyne, 1 for livox, 2 for 120*25 solid lidar -->
-    <xacro:arg name="lidar_type" default="2" />
+    <xacro:arg name="lidar_type" default="0" />
     <xacro:property name="lidar_type" value="$(arg lidar_type)" />
     <xacro:property name="base_x_size" value="0.9250000" />
@@ -36,9 +36,16 @@
     <xacro:if value="${lidar_type==0}">
         <!-- VLP16 激光雷达 -->
-        <xacro:include filename="$(find velodyne_description)/urdf/VLP-16.urdf.xacro"/>
+        <!-- <xacro:include filename="$(find velodyne_description)/urdf/VLP-16.urdf.xacro"/>
         <xacro:VLP-16 parent="support" name="lidar" topic="/scan" organize_cloud="${organize_cloud}"
         hz="10" samples="1800" max_range="150" gpu="${gpu}">
               <origin xyz="0 0 0" rpy="0 0 0" />
-        </xacro:VLP-16>
+        </xacro:VLP-16> -->
+        <xacro:include filename="$(find velodyne_description)/urdf/Lidar.urdf.xacro" />
+        <xacro:Lidar parent="support" name="lidar" topic="/scan" hz="10"
+            organize_cloud="${organize_cloud}" gpu="${gpu}"
+            samples="1800" min_horizonal_angle="${radians(-180.0)}" max_horizonal_angle="${radians(180.0)}"
+            lasers="16" min_vertical_angle="${radians(-15.0)}" max_vertical_angle="${radians(15.0)}">
+            <origin xyz="0 0 0" rpy="0 0 0" />
+        </xacro:Lidar>
     </xacro:if>
     <xacro:if value="${lidar_type==1}">

Commit message: add Readme and fix gitmodules bug

File: scout_gazebo/urdf/base.xacro (robot description, xacro)
@@ -4,5 +4,5 @@
     <!-- 属性封装 -->
     <!-- 0 for velodyne, 1 for livox, 2 for 120*25 solid lidar -->
-    <xacro:arg name="lidar_type" default="0" />
+    <xacro:arg name="lidar_type" default="1" />
     <xacro:property name="lidar_type" value="$(arg lidar_type)" />
     <xacro:property name="base_x_size" value="0.9250000" />
@@ -36,9 +36,4 @@
     <xacro:if value="${lidar_type==0}">
         <!-- VLP16 激光雷达 -->
-        <!-- <xacro:include filename="$(find velodyne_description)/urdf/VLP-16.urdf.xacro"/>
-        <xacro:VLP-16 parent="support" name="lidar" topic="/scan" organize_cloud="${organize_cloud}"
-        hz="10" samples="1800" max_range="150" gpu="${gpu}">
-              <origin xyz="0 0 0" rpy="0 0 0" />
-        </xacro:VLP-16> -->
         <xacro:include filename="$(find velodyne_description)/urdf/Lidar.urdf.xacro" />
         <xacro:Lidar parent="support" name="lidar" topic="/scan" hz="10"
